File: Placa/arion.sch (KiCad schematic (older format))
At the start: 33 parts, among them P1 CONN_01X03, P2 CONN_01X02, P3 CONN_01X06, SW1 SW_PUSH, SW2 SW_PUSH, SW3 SW_PUSH, U1 TCRT1000, U2 TCRT1000, U3 TCRT1000, U4 TCRT1000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

Commit message: Se cambiaron los errores que habia en la ultima version
Parts:
- D1, D2, D3: footprint LEDs:LED-0805 -> Resistors_SMD:R_0805_HandSoldering
- R1, R10, R11, R12, R13, R14, R15, R16, R17, R18, R2, R3, R4, R5, R6, R7, R8, R9: footprint Resistors_SMD:R_0805 -> Resistors_SMD:R_0805_HandSoldering
Changed lines of the file:
@@
 F 0 "R3" V 1680 2800 50  0000 C CNN
 F 1 "R" V 1600 2800 50  0000 C CNN
-F 2 "Resistors_SMD:R_0805" V 1530 2800 30  0001 C CNN
+F 2 "Resistors_SMD:R_0805_HandSoldering" V 1530 2800 30  0001 C CNN
 F 3 "" H 1600 2800 30  0000 C CNN
 	1    1600 2800
@@
 F 0 "R4" V 2280 2850 50  0000 C CNN
 F 1 "R" V 2200 2850 50  0000 C CNN
-F 2 "Resistors_SMD:R_0805" V 2130 2850 30  0001 C CNN
+F 2 "Resistors_SMD:R_0805_HandSoldering" V 2130 2850 30  0001 C CNN
 F 3 "" H 2200 2850 30  0000 C CNN
 	1    2200 2850
@@
 F 0 "R7" V 3530 2800 50  0000 C CNN
 F 1 "R" V 3450 2800 50  0000 C CNN
-F 2 "Resistors_SMD:R_0805" V 3380 2800 30  0001 C CNN
+F 2 "Resistors_SMD:R_0805_HandSoldering" V 3380 2800 30  0001 C CNN
 F 3 "" H 3450 2800 30  0000 C CNN
 	1    3450 2800
@@
 F 0 "R8" V 4130 2850 50  0000 C CNN
 F 1 "R" V 4050 2850 50  0000 C CNN
-F 2 "Resistors_SMD:R_0805" V 3980 2850 30  0001 C CNN
+F 2 "Resistors_SMD:R_0805_HandSoldering" V 3980 2850 30  0001 C CNN
 F 3 "" H 4050 2850 30  0000 C CNN
 	1    4050 2850
@@
 F 0 "R10" V 5380 2800 50  0000 C CNN
 F 1 "R" V 5300 2800 50  0000 C CNN
-F 2 "Resistors_SMD:R_0805" V 5230 2800 30  0001 C CNN
+F 2 "Resistors_SMD:R_0805_HandSoldering" V 5230 2800 30  0001 C CNN
 F 3 "" H 5300 2800 30  0000 C CNN
 	1    5300 2800
@@
 F 0 "R11" V 5980 2850 50  0000 C CNN
 F 1 "R" V 5900 2850 50  0000 C CNN
-F 2 "Resistors_SMD:R_0805" V 5830 2850 30  0001 C CNN
+F 2 "Resistors_SMD:R_0805_HandSoldering" V 5830 2850 30  0001 C CNN
 F 3 "" H 5900 2850 30  0000 C CNN
 	1    5900 2850
@@
 F 0 "R13" V 7230 2800 50  0000 C CNN
 F 1 "R" V 7150 2800 50  0000 C CNN
-F 2 "Resistors_SMD:R_0805" V 7080 2800 30  0001 C CNN
+F 2 "Resistors_SMD:R_0805_HandSoldering" V 7080 2800 30  0001 C CNN
 F 3 "" H 7150 2800 30  0000 C CNN
 	1    7150 2800
@@
 F 0 "R14" V 7830 2850 50  0000 C CNN
 F 1 "R" V 7750 2850 50  0000 C CNN
-F 2 "Resistors_SMD:R_0805" V 7680 2850 30  0001 C CNN
+F 2 "Resistors_SMD:R_0805_HandSoldering" V 7680 2850 30  0001 C CNN
 F 3 "" H 7750 2850 30  0000 C CNN
 	1    7750 2850
@@
 F 0 "R16" V 9030 2800 50  0000 C CNN
 F 1 "R" V 8950 2800 50  0000 C CNN
-F 2 "Resistors_SMD:R_0805" V 8880 2800 30  0001 C CNN
+F 2 "Resistors_SMD:R_0805_HandSoldering" V 8880 2800 30  0001 C CNN
 F 3 "" H 8950 2800 30  0000 C CNN
 	1    8950 2800
@@
 F 0 "R17" V 9630 2850 50  0000 C CNN
 F 1 "R" V 9550 2850 50  0000 C CNN
-F 2 "Resistors_SMD:R_0805" V 9480 2850 30  0001 C CNN
+F 2 "Resistors_SMD:R_0805_HandSoldering" V 9480 2850 30  0001 C CNN
 F 3 "" H 9550 2850 30  0000 C CNN
 	1    9550 2850
@@
 F 0 "R5" V 3430 900 50  0000 C CNN
 F 1 "R" V 3350 900 50  0000 C CNN
-F 2 "Resistors_SMD:R_0805" V 3280 900 30  0001 C CNN
+F 2 "Resistors_SMD:R_0805_HandSoldering" V 3280 900 30  0001 C CNN
 F 3 "" H 3350 900 30  0000 C CNN
 	1    3350 900
@@
 F 0 "R6" V 3430 1350 50  0000 C CNN
 F 1 "R" V 3350 1350 50  0000 C CNN
-F 2 "Resistors_SMD:R_0805" V 3280 1350 30  0001 C CNN
+F 2 "Resistors_SMD:R_0805_HandSoldering" V 3280 1350 30  0001 C CNN
 F 3 "" H 3350 1350 30  0000 C CNN
 	1    3350 1350
@@
 F 0 "R12" V 7130 4500 50  0000 C CNN
 F 1 "R" V 7050 4500 50  0000 C CNN
-F 2 "Resistors_SMD:R_0805" V 6980 4500 30  0001 C CNN
+F 2 "Resistors_SMD:R_0805_HandSoldering" V 6980 4500 30  0001 C CNN
 F 3 "" H 7050 4500 30  0000 C CNN
 	1    7050 4500
@@
 F 0 "R15" V 7880 4500 50  0000 C CNN
 F 1 "R" V 7800 4500 50  0000 C CNN
-F 2 "Resistors_SMD:R_0805" V 7730 4500 30  0001 C CNN
+F 2 "Resistors_SMD:R_0805_HandSoldering" V 7730 4500 30  0001 C CNN
 F 3 "" H 7800 4500 30  0000 C CNN
 	1    7800 4500
@@
 F 0 "R18" V 8630 4500 50  0000 C CNN
 F 1 "R" V 8550 4500 50  0000 C CNN
-F 2 "Resistors_SMD:R_0805" V 8480 4500 30  0001 C CNN
+F 2 "Resistors_SMD:R_0805_HandSoldering" V 8480 4500 30  0001 C CNN
 F 3 "" H 8550 4500 30  0000 C CNN
 	1    8550 4500
@@
 F 0 "D1" H 1250 5800 50  0000 C CNN
 F 1 "LED" H 1250 5600 50  0000 C CNN
-F 2 "LEDs:LED-0805" H 1250 5700 60  0001 C CNN
+F 2 "Resistors_SMD:R_0805_HandSoldering" H 1250 5700 60  0001 C CNN
 F 3 "" H 1250 5700 60  0000 C CNN
 	1    1250 5700
@@
 F 0 "D2" H 1550 5800 50  0000 C CNN
 F 1 "LED" H 1550 5600 50  0000 C CNN
-F 2 "LEDs:LED-0805" H 1550 5700 60  0001 C CNN
+F 2 "Resistors_SMD:R_0805_HandSoldering" H 1550 5700 60  0001 C CNN
 F 3 "" H 1550 5700 60  0000 C CNN
 	1    1550 5700
@@
 F 0 "R1" V 1330 6100 50  0000 C CNN
 F 1 "R" V 1250 6100 50  0000 C CNN
-F 2 "Resistors_SMD:R_0805" V 1180 6100 30  0001 C CNN
+F 2 "Resistors_SMD:R_0805_HandSoldering" V 1180 6100 30  0001 C CNN
 F 3 "" H 1250 6100 30  0000 C CNN
 	1    1250 6100
@@
 F 0 "R2" V 1630 6100 50  0000 C CNN
 F 1 "R" V 1550 6100 50  0000 C CNN
-F 2 "Resistors_SMD:R_0805" V 1480 6100 30  0001 C CNN
+F 2 "Resistors_SMD:R_0805_HandSoldering" V 1480 6100 30  0001 C CNN
 F 3 "" H 1550 6100 30  0000 C CNN
 	1    1550 6100
@@
 F 0 "D3" H 4650 5650 50  0000 C CNN
 F 1 "LED" H 4650 5450 50  0000 C CNN
-F 2 "LEDs:LED-0805" H 4650 5550 60  0001 C CNN
+F 2 "Resistors_SMD:R_0805_HandSoldering" H 4650 5550 60  0001 C CNN
 F 3 "" H 4650 5550 60  0000 C CNN
 	1    4650 5550
@@
 F 0 "R9" V 4730 5950 50  0000 C CNN
 F 1 "R" V 4650 5950 50  0000 C CNN
-F 2 "Resistors_SMD:R_0805" V 4580 5950 30  0001 C CNN
+F 2 "Resistors_SMD:R_0805_HandSoldering" V 4580 5950 30  0001 C CNN
 F 3 "" H 4650 5950 30  0000 C CNN
 	1    4650 5950
