File: Placa/Motores.sch (KiCad schematic (older format))
At the start: 15 parts, among them U1 DVR8833, U2 DVR8833

Commit message: Avances sobre la placa.
Parts:
- removed P? (x2): CONN_01X02, symbol CONN_01X02
- C2, C3, C4, C5: footprint ~ -> Capacitors_SMD:C_0805_HandSoldering
- C6: renamed from C?; value CP -> 10uF; footprint (none) -> Capacitors_ThroughHole:C_Radial_D5_L11_P2.5
- D1: footprint ~ -> LEDs:LED_0805
- P4, P6: renamed from P?; footprint (none) -> Pin_Headers:Pin_Header_Straight_1x01
- P5, P7: renamed from P?; footprint (none) -> Pin_Headers:Pin_Header_Straight_1x02
- R1: footprint ~ -> Resistors_SMD:R_0805
- U1, U2: footprint MODULE -> Housings_SSOP:TSSOP-16_4.4x5mm_Pitch0.65mm
Connections:
- wire segments 67 -> 59
Changed lines of the file:
@@
 F 0 "U1" H 4400 3700 50  0000 C CNN
 F 1 "DVR8833" H 4400 3900 50  0000 C CNN
-F 2 "MODULE" H 4400 3800 50  0001 C CNN
+F 2 "Housings_SSOP:TSSOP-16_4.4x5mm_Pitch0.65mm" H 4400 3800 50  0001 C CNN
 F 3 "DOCUMENTATION" H 4400 3800 50  0001 C CNN
 	1    4400 3800
@@
 F 0 "U2" H 7150 3700 50  0000 C CNN
 F 1 "DVR8833" H 7150 3900 50  0000 C CNN
-F 2 "MODULE" H 7150 3800 50  0001 C CNN
+F 2 "Housings_SSOP:TSSOP-16_4.4x5mm_Pitch0.65mm" H 7150 3800 50  0001 C CNN
 F 3 "DOCUMENTATION" H 7150 3800 50  0001 C CNN
 	1    7150 3800
@@
 F 0 "C2" H 4350 2250 40  0000 L CNN
 F 1 "0.01u" H 4356 2065 40  0000 L CNN
-F 2 "~" H 4388 2000 30  0000 C CNN
+F 2 "Capacitors_SMD:C_0805_HandSoldering" H 4388 2000 30  0000 C CNN
 F 3 "~" H 4350 2150 60  0000 C CNN
 	1    4350 2150
@@
 F 0 "C4" H 5250 2300 40  0000 L CNN
 F 1 "2.2u" H 5256 2115 40  0000 L CNN
-F 2 "~" H 5288 2050 30  0000 C CNN
+F 2 "Capacitors_SMD:C_0805_HandSoldering" H 5288 2050 30  0000 C CNN
 F 3 "~" H 5250 2200 60  0000 C CNN
 	1    5250 2200
@@
 F 0 "C5" H 5700 2300 40  0000 L CNN
 F 1 "2.2u" H 5706 2115 40  0000 L CNN
-F 2 "~" H 5738 2050 30  0000 C CNN
+F 2 "Capacitors_SMD:C_0805_HandSoldering" H 5738 2050 30  0000 C CNN
 F 3 "~" H 5700 2200 60  0000 C CNN
 	1    5700 2200
@@
 F 0 "C3" H 4750 2250 40  0000 L CNN
 F 1 "0.01u" H 4756 2065 40  0000 L CNN
-F 2 "~" H 4788 2000 30  0000 C CNN
+F 2 "Capacitors_SMD:C_0805_HandSoldering" H 4788 2000 30  0000 C CNN
 F 3 "~" H 4750 2150 60  0000 C CNN
 	1    4750 2150
@@
 F 0 "R1" V 7630 1950 40  0000 C CNN
 F 1 "1k" V 7557 1951 40  0000 C CNN
-F 2 "~" V 7480 1950 30  0000 C CNN
+F 2 "Resistors_SMD:R_0805" V 7480 1950 30  0001 C CNN
 F 3 "~" H 7550 1950 30  0000 C CNN
 	1    7550 1950
@@
 F 0 "D1" H 7550 2600 50  0000 C CNN
 F 1 "LED" H 7550 2400 50  0000 C CNN
-F 2 "~" H 7550 2500 60  0000 C CNN
+F 2 "LEDs:LED_0805" H 7550 2500 60  0001 C CNN
 F 3 "~" H 7550 2500 60  0000 C CNN
 	1    7550 2500
@@
 $EndComp
 $Comp
-L GND #PWR01
+L GND #PWR037
 U 1 1 55EB036E
 P 3100 3700
-F 0 "#PWR01" H 3100 3700 30  0001 C CNN
+F 0 "#PWR037" H 3100 3700 30  0001 C CNN
 F 1 "GND" H 3100 3630 30  0001 C CNN
 F 2 "" H 3100 3700 60  0000 C CNN
@@
 $EndComp
 $Comp
-L GND #PWR02
+L GND #PWR038
 U 1 1 55EB037B
 P 3100 4000
-F 0 "#PWR02" H 3100 4000 30  0001 C CNN
+F 0 "#PWR038" H 3100 4000 30  0001 C CNN
 F 1 "GND" H 3100 3930 30  0001 C CNN
 F 2 "" H 3100 4000 60  0000 C CNN
@@
 $EndComp
 $Comp
-L GND #PWR03
+L GND #PWR039
 U 1 1 55EB0384
 P 5850 3700
-F 0 "#PWR03" H 5850 3700 30  0001 C CNN
+F 0 "#PWR039" H 5850 3700 30  0001 C CNN
 F 1 "GND" H 5850 3630 30  0001 C CNN
 F 2 "" H 5850 3700 60  0000 C CNN
@@
 $EndComp
 $Comp
-L GND #PWR04
+L GND #PWR040
 U 1 1 55EB0393
 P 5850 4000
-F 0 "#PWR04" H 5850 4000 30  0001 C CNN
+F 0 "#PWR040" H 5850 4000 30  0001 C CNN
 F 1 "GND" H 5850 3930 30  0001 C CNN
 F 2 "" H 5850 4000 60  0000 C CNN
@@
 $EndComp
 $Comp
-L GND #PWR05
+L GND #PWR041
 U 1 1 55EB047B
 P 5600 3800
-F 0 "#PWR05" H 5600 3800 30  0001 C CNN
+F 0 "#PWR041" H 5600 3800 30  0001 C CNN
 F 1 "GND" H 5600 3730 30  0001 C CNN
 F 2 "" H 5600 3800 60  0000 C CNN
@@
 $EndComp
 $Comp
-L GND #PWR06
+L GND #PWR042
 U 1 1 55EB0487
 P 8550 3800
-F 0 "#PWR06" H 8550 3800 30  0001 C CNN
+F 0 "#PWR042" H 8550 3800 30  0001 C CNN
 F 1 "GND" H 8550 3730 30  0001 C CNN
 F 2 "" H 8550 3800 60  0000 C CNN
@@
 	5600 3750 5600 3800
 Wire Wire Line
-	5150 3950 5200 3950
+	5150 3950 5450 3950
 Wire Wire Line
 	6350 3550 6400 3550
@@
 	7900 3850 7950 3850
 Wire Wire Line
-	7900 3950 7950 3950
+	7900 3950 8250 3950
 Wire Wire Line
 	3900 1950 4750 1950
@@
 	4350 2300 4350 2450
 $Comp
-L GND #PWR07
+L GND #PWR043
 U 1 1 55EB1201
 P 3900 2450
-F 0 "#PWR07" H 3900 2450 30  0001 C CNN
+F 0 "#PWR043" H 3900 2450 30  0001 C CNN
 F 1 "GND" H 3900 2380 30  0001 C CNN
 F 2 "" H 3900 2450 60  0000 C CNN
@@
 	1    0    0    -1
 $EndComp
-Wire Wire Line
-	3250 2000 3300 2000
-Wire Wire Line
-	3250 2200 3300 2200
-Wire Wire Line
-	3250 2450 3300 2450
-Wire Wire Line
-	3250 2650 3300 2650
-$Comp
-L GND #PWR08
+$Comp
+L GND #PWR044
 U 1 1 55EB12DF
 P 5250 2450
-F 0 "#PWR08" H 5250 2450 30  0001 C CNN
+F 0 "#PWR044" H 5250 2450 30  0001 C CNN
 F 1 "GND" H 5250 2380 30  0001 C CNN
 F 2 "" H 5250 2450 60  0000 C CNN
@@
 $EndComp
 $Comp
-L GND #PWR09
+L GND #PWR045
 U 1 1 55EB12E5
 P 5700 2450
-F 0 "#PWR09" H 5700 2450 30  0001 C CNN
+F 0 "#PWR045" H 5700 2450 30  0001 C CNN
 F 1 "GND" H 5700 2380 30  0001 C CNN
 F 2 "" H 5700 2450 60  0000 C CNN
@@
 	3900 2300 3900 2450
 $Comp
-L GND #PWR011
+L GND #PWR046
 U 1 1 55EB18C4
 P 7550 2800
-F 0 "#PWR011" H 7550 2800 30  0001 C CNN
+F 0 "#PWR046" H 7550 2800 30  0001 C CNN
 F 1 "GND" H 7550 2730 30  0001 C CNN
 F 2 "" H 7550 2800 60  0000 C CNN
@@
 	7550 1650 7550 1800
 $Comp
-L CONN_01X01 P?
+L CONN_01X01 P4
 U 1 1 571ABD6A
 P 2850 4150
-F 0 "P?" H 2850 4250 50  0000 C CNN
+F 0 "P4" H 2850 4250 50  0000 C CNN
 F 1 "CONN_01X01" V 2950 4150 50  0000 C CNN
-F 2 "" H 2850 4150 50  0000 C CNN
+F 2 "Pin_Headers:Pin_Header_Straight_1x01" H 2850 4150 50  0001 C CNN
 F 3 "" H 2850 4150 50  0000 C CNN
 	1    2850 4150
@@
 $EndComp
 $Comp
-L CONN_01X01 P?
+L CONN_01X01 P6
 U 1 1 571ABE3D
 P 5700 4150
-F 0 "P?" H 5700 4250 50  0000 C CNN
+F 0 "P6" H 5700 4250 50  0000 C CNN
 F 1 "CONN_01X01" V 5800 4150 50  0000 C CNN
-F 2 "" H 5700 4150 50  0000 C CNN
+F 2 "Pin_Headers:Pin_Header_Straight_1x01" H 5700 4150 50  0001 C CNN
 F 3 "" H 5700 4150 50  0000 C CNN
 	1    5700 4150
@@
 $EndComp
 $Comp
-L CONN_01X02 P?
+L CONN_01X02 P7
 U 1 1 571ABEF8
 P 5950 3200
-F 0 "P?" H 5950 3350 50  0000 C CNN
+F 0 "P7" H 5950 3350 50  0000 C CNN
 F 1 "CONN_01X02" V 6050 3200 50  0000 C CNN
-F 2 "" H 5950 3200 50  0000 C CNN
+F 2 "Pin_Headers:Pin_Header_Straight_1x02" H 5950 3200 50  0001 C CNN
 F 3 "" H 5950 3200 50  0000 C CNN
 	1    5950 3200
@@
 $EndComp
 $Comp
-L CONN_01X02 P?
+L CONN_01X02 P5
 U 1 1 571ABF5C
 P 3200 3200
-F 0 "P?" H 3200 3350 50  0000 C CNN
+F 0 "P5" H 3200 3350 50  0000 C CNN
 F 1 "CONN_01X02" V 3300 3200 50  0000 C CNN
-F 2 "" H 3200 3200 50  0000 C CNN
+F 2 "Pin_Headers:Pin_Header_Straight_1x02" H 3200 3200 50  0001 C CNN
 F 3 "" H 3200 3200 50  0000 C CNN
 	1    3200 3200
@@
 	4750 1950 4750 2000
 $Comp
-L CONN_01X02 P?
-U 1 1 571AC5DD
-P 3500 2100
-F 0 "P?" H 3500 2250 50  0000 C CNN
-F 1 "CONN_01X02" V 3600 2100 50  0000 C CNN
-F 2 "" H 3500 2100 50  0000 C CNN
-F 3 "" H 3500 2100 50  0000 C CNN
-	1    3500 2100
-	1    0    0    -1
-$EndComp
-Wire Wire Line
-	3300 2000 3300 2050
-Wire Wire Line
-	3300 2200 3300 2150
-$Comp
-L CONN_01X02 P?
-U 1 1 571AC6E1
-P 3500 2550
-F 0 "P?" H 3500 2700 50  0000 C CNN
-F 1 "CONN_01X02" V 3600 2550 50  0000 C CNN
-F 2 "" H 3500 2550 50  0000 C CNN
-F 3 "" H 3500 2550 50  0000 C CNN
-	1    3500 2550
-	1    0    0    -1
-$EndComp
-Wire Wire Line
-	3300 2450 3300 2500
-Wire Wire Line
-	3300 2650 3300 2600
-$Comp
-L CP C?
+L CP C6
 U 1 1 571AC7CC
 P 3900 2150
-F 0 "C?" H 3925 2250 50  0000 L CNN
-F 1 "CP" H 3925 2050 50  0000 L CNN
-F 2 "" H 3938 2000 50  0000 C CNN
+F 0 "C6" H 3925 2250 50  0000 L CNN
+F 1 "10uF" H 3925 2050 50  0000 L CNN
+F 2 "Capacitors_ThroughHole:C_Radial_D5_L11_P2.5" H 3938 2000 50  0001 C CNN
 F 3 "" H 3900 2150 50  0000 C CNN
 	1    3900 2150
@@
 Text HLabel 7950 3850 2    60   Input ~ 0
 VM
-Text HLabel 7950 3950 2    60   Input ~ 0
-M2VCP
 Text HLabel 7950 4050 2    60   Input ~ 0
 M2IN2
@@
 Text HLabel 5200 4150 2    60   Input ~ 0
 M1IN1
-Text HLabel 5200 3950 2    60   Input ~ 0
-M1VCP
 Text HLabel 3600 3550 0    60   Input ~ 0
 M1OUT1
@@
 Text HLabel 7550 1650 0    60   Input ~ 0
 VM
-Text HLabel 3250 2000 0    60   Input ~ 0
-M1OUT1
-Text HLabel 3250 2200 0    60   Input ~ 0
-M1OUT2
-Text HLabel 3250 2450 0    60   Input ~ 0
-M2OUT1
-Text HLabel 3250 2650 0    60   Input ~ 0
-M2OUT2
 Text HLabel 5250 1950 0    60   Input ~ 0
 M1VINT
 Text HLabel 5700 1950 0    60   Input ~ 0
 M2VINT
-Text HLabel 4750 2450 0    60   Input ~ 0
+Text HLabel 4550 1850 0    60   Input ~ 0
+VM
+Text HLabel 3000 3450 0    60   Input ~ 0
+VM
+Text Label 4350 2450 2    60   ~ 0
+M1VCP
+Text Label 5450 3950 2    60   ~ 0
+M1VCP
+Text Label 8250 3950 2    60   ~ 0
 M2VCP
-Text HLabel 4350 2450 0    60   Input ~ 0
-M1VCP
-Text HLabel 4550 1850 0    60   Input ~ 0
-VM
-Text HLabel 3000 3450 0    60   Input ~ 0
-VM
+Text Label 4750 2450 2    60   ~ 0
+M2VCP
 $EndSCHEMATC

Commit message: Más avances en placa. Ignorados archivos bak.
Falta corregir algunas cosas en el esquemático, relacionado con los motores. El pcb está apenas empezado.
Se ignoraron los archivos bak y cache de kicad.
Parts:
- removed P5, P7: CONN_01X02, Pin_Headers:Pin_Header_Straight_1x02, symbol CONN_01X02
Connections:
- wire segments 59 -> 53
Changed lines of the file:
@@
 LIBS:reg_204-5
 LIBS:DVR8833
-LIBS:placa-cache
 EELAYER 25 0
 EELAYER END
@@
 $EndComp
 $Comp
-L GND #PWR037
+L GND #PWR039
 U 1 1 55EB036E
 P 3100 3700
-F 0 "#PWR037" H 3100 3700 30  0001 C CNN
+F 0 "#PWR039" H 3100 3700 30  0001 C CNN
 F 1 "GND" H 3100 3630 30  0001 C CNN
 F 2 "" H 3100 3700 60  0000 C CNN
@@
 $EndComp
 $Comp
-L GND #PWR038
+L GND #PWR040
 U 1 1 55EB037B
 P 3100 4000
-F 0 "#PWR038" H 3100 4000 30  0001 C CNN
+F 0 "#PWR040" H 3100 4000 30  0001 C CNN
 F 1 "GND" H 3100 3930 30  0001 C CNN
 F 2 "" H 3100 4000 60  0000 C CNN
@@
 $EndComp
 $Comp
-L GND #PWR039
+L GND #PWR041
 U 1 1 55EB0384
 P 5850 3700
-F 0 "#PWR039" H 5850 3700 30  0001 C CNN
+F 0 "#PWR041" H 5850 3700 30  0001 C CNN
 F 1 "GND" H 5850 3630 30  0001 C CNN
 F 2 "" H 5850 3700 60  0000 C CNN
@@
 $EndComp
 $Comp
-L GND #PWR040
+L GND #PWR042
 U 1 1 55EB0393
 P 5850 4000
-F 0 "#PWR040" H 5850 4000 30  0001 C CNN
+F 0 "#PWR042" H 5850 4000 30  0001 C CNN
 F 1 "GND" H 5850 3930 30  0001 C CNN
 F 2 "" H 5850 4000 60  0000 C CNN
@@
 $EndComp
 $Comp
-L GND #PWR041
+L GND #PWR043
 U 1 1 55EB047B
 P 5600 3800
-F 0 "#PWR041" H 5600 3800 30  0001 C CNN
+F 0 "#PWR043" H 5600 3800 30  0001 C CNN
 F 1 "GND" H 5600 3730 30  0001 C CNN
 F 2 "" H 5600 3800 60  0000 C CNN
@@
 $EndComp
 $Comp
-L GND #PWR042
+L GND #PWR044
 U 1 1 55EB0487
 P 8550 3800
-F 0 "#PWR042" H 8550 3800 30  0001 C CNN
+F 0 "#PWR044" H 8550 3800 30  0001 C CNN
 F 1 "GND" H 8550 3730 30  0001 C CNN
 F 2 "" H 8550 3800 60  0000 C CNN
@@
 	4350 2300 4350 2450
 $Comp
-L GND #PWR043
+L GND #PWR045
 U 1 1 55EB1201
 P 3900 2450
-F 0 "#PWR043" H 3900 2450 30  0001 C CNN
+F 0 "#PWR045" H 3900 2450 30  0001 C CNN
 F 1 "GND" H 3900 2380 30  0001 C CNN
 F 2 "" H 3900 2450 60  0000 C CNN
@@
 $EndComp
 $Comp
-L GND #PWR044
+L GND #PWR046
 U 1 1 55EB12DF
 P 5250 2450
-F 0 "#PWR044" H 5250 2450 30  0001 C CNN
+F 0 "#PWR046" H 5250 2450 30  0001 C CNN
 F 1 "GND" H 5250 2380 30  0001 C CNN
 F 2 "" H 5250 2450 60  0000 C CNN
@@
 $EndComp
 $Comp
-L GND #PWR045
+L GND #PWR047
 U 1 1 55EB12E5
 P 5700 2450
-F 0 "#PWR045" H 5700 2450 30  0001 C CNN
+F 0 "#PWR047" H 5700 2450 30  0001 C CNN
 F 1 "GND" H 5700 2380 30  0001 C CNN
 F 2 "" H 5700 2450 60  0000 C CNN
@@
 	5700 2350 5700 2450
 Wire Wire Line
-	6000 3450 6400 3450
-Wire Wire Line
-	3250 3450 3650 3450
-Wire Wire Line
-	3000 3450 3150 3450
+	5850 3450 6400 3450
+Wire Wire Line
+	3000 3450 3650 3450
 Wire Wire Line
 	3050 4150 3650 4150
@@
 	3900 2300 3900 2450
 $Comp
-L GND #PWR046
+L GND #PWR048
 U 1 1 55EB18C4
 P 7550 2800
-F 0 "#PWR046" H 7550 2800 30  0001 C CNN
+F 0 "#PWR048" H 7550 2800 30  0001 C CNN
 F 1 "GND" H 7550 2730 30  0001 C CNN
 F 2 "" H 7550 2800 60  0000 C CNN
@@
 	-1   0    0    1
 $EndComp
-$Comp
-L CONN_01X02 P7
-U 1 1 571ABEF8
-P 5950 3200
-F 0 "P7" H 5950 3350 50  0000 C CNN
-F 1 "CONN_01X02" V 6050 3200 50  0000 C CNN
-F 2 "Pin_Headers:Pin_Header_Straight_1x02" H 5950 3200 50  0001 C CNN
-F 3 "" H 5950 3200 50  0000 C CNN
-	1    5950 3200
-	0    -1   -1   0
-$EndComp
-$Comp
-L CONN_01X02 P5
-U 1 1 571ABF5C
-P 3200 3200
-F 0 "P5" H 3200 3350 50  0000 C CNN
-F 1 "CONN_01X02" V 3300 3200 50  0000 C CNN
-F 2 "Pin_Headers:Pin_Header_Straight_1x02" H 3200 3200 50  0001 C CNN
-F 3 "" H 3200 3200 50  0000 C CNN
-	1    3200 3200
-	0    -1   -1   0
-$EndComp
-Wire Wire Line
-	3150 3450 3150 3400
-Wire Wire Line
-	3250 3400 3250 3450
-Wire Wire Line
-	5900 3450 5900 3400
-Wire Wire Line
-	6000 3400 6000 3450
 Wire Wire Line
 	4350 2000 4350 1950
@@
 Text HLabel 5850 3450 0    60   Input ~ 0
 VM
-Wire Wire Line
-	5850 3450 5900 3450
 Text HLabel 6350 3550 0    60   Input ~ 0
 M2OUT1

Commit message: Placa: ajustes al sch del puente H.
Parts:
- removed D1: LED, LEDs:LED_0805, symbol LED
- removed P4, P6: CONN_01X01, Pin_Headers:Pin_Header_Straight_1x01, symbol CONN_01X01
- removed R1: 1k, Resistors_SMD:R_0805, symbol R
- added R? (x2): 200m, symbol R
- added R? (x2): 50k, symbol R
Connections:
- net labels added: xISEN1, xISEN2
- wire segments 53 -> 54
- no-connect marks 0 -> 2
Changed lines of the file:
@@
-$EndComp
-$Comp
-L R R1
-U 1 1 55EAFB5A
-P 7550 1950
-F 0 "R1" V 7630 1950 40  0000 C CNN
-F 1 "1k" V 7557 1951 40  0000 C CNN
-F 2 "Resistors_SMD:R_0805" V 7480 1950 30  0001 C CNN
-F 3 "~" H 7550 1950 30  0000 C CNN
-	1    7550 1950
-	1    0    0    -1
-$EndComp
-$Comp
-L LED D1
-U 1 1 55EAFB78
-P 7550 2500
-F 0 "D1" H 7550 2600 50  0000 C CNN
-F 1 "LED" H 7550 2400 50  0000 C CNN
-F 2 "LEDs:LED_0805" H 7550 2500 60  0001 C CNN
-F 3 "~" H 7550 2500 60  0000 C CNN
-	1    7550 2500
-	0    -1   -1   0
-$EndComp
-$Comp
-L GND #PWR039
-U 1 1 55EB036E
-P 3100 3700
-F 0 "#PWR039" H 3100 3700 30  0001 C CNN
-F 1 "GND" H 3100 3630 30  0001 C CNN
-F 2 "" H 3100 3700 60  0000 C CNN
-F 3 "" H 3100 3700 60  0000 C CNN
-	1    3100 3700
-	1    0    0    -1
-$EndComp
-$Comp
-L GND #PWR040
-U 1 1 55EB037B
-P 3100 4000
-F 0 "#PWR040" H 3100 4000 30  0001 C CNN
-F 1 "GND" H 3100 3930 30  0001 C CNN
-F 2 "" H 3100 4000 60  0000 C CNN
-F 3 "" H 3100 4000 60  0000 C CNN
-	1    3100 4000
-	1    0    0    -1
-$EndComp
-$Comp
-L GND #PWR041
-U 1 1 55EB0384
-P 5850 3700
-F 0 "#PWR041" H 5850 3700 30  0001 C CNN
-F 1 "GND" H 5850 3630 30  0001 C CNN
-F 2 "" H 5850 3700 60  0000 C CNN
-F 3 "" H 5850 3700 60  0000 C CNN
-	1    5850 3700
-	1    0    0    -1
-$EndComp
-$Comp
-L GND #PWR042
-U 1 1 55EB0393
-P 5850 4000
-F 0 "#PWR042" H 5850 4000 30  0001 C CNN
-F 1 "GND" H 5850 3930 30  0001 C CNN
-F 2 "" H 5850 4000 60  0000 C CNN
-F 3 "" H 5850 4000 60  0000 C CNN
-	1    5850 4000
-	1    0    0    -1
 $EndComp
 $Comp
@@
 	3600 3550 3650 3550
 Wire Wire Line
-	3650 3650 3100 3650
-Wire Wire Line
-	3100 3650 3100 3700
-Wire Wire Line
 	3600 3750 3650 3750
 Wire Wire Line
 	3600 3850 3650 3850
 Wire Wire Line
-	3650 3950 3100 3950
-Wire Wire Line
-	3100 3950 3100 4000
-Wire Wire Line
 	3600 4050 3650 4050
 Wire Wire Line
@@
 	6350 3550 6400 3550
 Wire Wire Line
-	6400 3650 5850 3650
-Wire Wire Line
-	5850 3650 5850 3700
-Wire Wire Line
 	6400 3750 6350 3750
 Wire Wire Line
 	6400 3850 6350 3850
-Wire Wire Line
-	6400 3950 5850 3950
-Wire Wire Line
-	5850 3950 5850 4000
 Wire Wire Line
 	6350 4050 6400 4050
@@
 	5700 2350 5700 2450
 Wire Wire Line
-	5850 3450 6400 3450
-Wire Wire Line
-	3000 3450 3650 3450
-Wire Wire Line
-	3050 4150 3650 4150
-Wire Wire Line
-	5900 4150 6400 4150
-Wire Wire Line
 	7950 3650 7900 3650
 Wire Wire Line
@@
 Wire Wire Line
 	3900 2300 3900 2450
-$Comp
-L GND #PWR048
-U 1 1 55EB18C4
-P 7550 2800
-F 0 "#PWR048" H 7550 2800 30  0001 C CNN
-F 1 "GND" H 7550 2730 30  0001 C CNN
-F 2 "" H 7550 2800 60  0000 C CNN
-F 3 "" H 7550 2800 60  0000 C CNN
-	1    7550 2800
-	1    0    0    -1
-$EndComp
-Wire Wire Line
-	7550 2100 7550 2300
-Wire Wire Line
-	7550 2700 7550 2800
-Wire Wire Line
-	7550 1650 7550 1800
-$Comp
-L CONN_01X01 P4
-U 1 1 571ABD6A
-P 2850 4150
-F 0 "P4" H 2850 4250 50  0000 C CNN
-F 1 "CONN_01X01" V 2950 4150 50  0000 C CNN
-F 2 "Pin_Headers:Pin_Header_Straight_1x01" H 2850 4150 50  0001 C CNN
-F 3 "" H 2850 4150 50  0000 C CNN
-	1    2850 4150
-	-1   0    0    1
-$EndComp
-$Comp
-L CONN_01X01 P6
-U 1 1 571ABE3D
-P 5700 4150
-F 0 "P6" H 5700 4250 50  0000 C CNN
-F 1 "CONN_01X01" V 5800 4150 50  0000 C CNN
-F 2 "Pin_Headers:Pin_Header_Straight_1x01" H 5700 4150 50  0001 C CNN
-F 3 "" H 5700 4150 50  0000 C CNN
-	1    5700 4150
-	-1   0    0    1
-$EndComp
 Wire Wire Line
 	4350 2000 4350 1950
@@
 Text HLabel 7950 4150 2    60   Input ~ 0
 M2IN1
-Text HLabel 5850 3450 0    60   Input ~ 0
+Text HLabel 5850 3300 0    60   Input ~ 0
 VM
 Text HLabel 6350 3550 0    60   Input ~ 0
@@
 Text HLabel 3600 4050 0    60   Input ~ 0
 M1OUT1
-Text HLabel 7550 1650 0    60   Input ~ 0
-VM
 Text HLabel 5250 1950 0    60   Input ~ 0
 M1VINT
@@
 Text HLabel 4550 1850 0    60   Input ~ 0
 VM
-Text HLabel 3000 3450 0    60   Input ~ 0
+Text HLabel 3050 3300 0    60   Input ~ 0
 VM
 Text Label 4350 2450 2    60   ~ 0
@@
 Text Label 4750 2450 2    60   ~ 0
 M2VCP
+Text Label 1350 2500 0    60   ~ 0
+xISEN1
+Wire Wire Line
+	3650 3650 3600 3650
+Wire Wire Line
+	3650 3950 3600 3950
+Text Label 3600 3650 2    60   ~ 0
+xISEN1
+Text Label 3600 3950 2    60   ~ 0
+xISEN1
+$Comp
+L R R?
+U 1 1 5748FFC9
+P 1850 2500
+F 0 "R?" V 1930 2500 50  0000 C CNN
+F 1 "200m" V 1850 2500 50  0000 C CNN
+F 2 "" V 1780 2500 50  0000 C CNN
+F 3 "" H 1850 2500 50  0000 C CNN
+	1    1850 2500
+	0    1    1    0
+$EndComp
+Wire Wire Line
+	1350 2500 1700 2500
+Wire Wire Line
+	2000 2500 2150 2500
+Wire Wire Line
+	2150 2500 2150 2550
+$Comp
+L GND #PWR?
+U 1 1 5749021E
+P 2150 2550
+F 0 "#PWR?" H 2150 2300 50  0001 C CNN
+F 1 "GND" H 2150 2400 50  0000 C CNN
+F 2 "" H 2150 2550 50  0000 C CNN
+F 3 "" H 2150 2550 50  0000 C CNN
+	1    2150 2550
+	1    0    0    -1
+$EndComp
+Text Label 1350 2950 0    60   ~ 0
+xISEN2
+$Comp
+L R R?
+U 1 1 574909EB
+P 1850 2950
+F 0 "R?" V 1930 2950 50  0000 C CNN
+F 1 "200m" V 1850 2950 50  0000 C CNN
+F 2 "" V 1780 2950 50  0000 C CNN
+F 3 "" H 1850 2950 50  0000 C CNN
+	1    1850 2950
+	0    1    1    0
+$EndComp
+Wire Wire Line
+	1350 2950 1700 2950
+Wire Wire Line
+	2000 2950 2150 2950
+Wire Wire Line
+	2150 2950 2150 3000
+$Comp
+L GND #PWR?
+U 1 1 574909F4
+P 2150 3000
+F 0 "#PWR?" H 2150 2750 50  0001 C CNN
+F 1 "GND" H 2150 2850 50  0000 C CNN
+F 2 "" H 2150 3000 50  0000 C CNN
+F 3 "" H 2150 3000 50  0000 C CNN
+	1    2150 3000
+	1    0    0    -1
+$EndComp
+Wire Wire Line
+	6350 3650 6400 3650
+Text Label 6350 3650 2    60   ~ 0
+xISEN2
+Text Label 6400 3950 2    60   ~ 0
+xISEN2
+NoConn ~ 3650 4150
+NoConn ~ 6400 4150
+Wire Wire Line
+	3700 3450 3650 3450
+Wire Wire Line
+	3650 3450 3650 3300
+Wire Wire Line
+	3650 3300 3500 3300
+$Comp
+L R R?
+U 1 1 57492D3E
+P 3350 3300
+F 0 "R?" V 3430 3300 50  0000 C CNN
+F 1 "50k" V 3350 3300 50  0000 C CNN
+F 2 "" V 3280 3300 50  0000 C CNN
+F 3 "" H 3350 3300 50  0000 C CNN
+	1    3350 3300
+	0    1    1    0
+$EndComp
+$Comp
+L R R?
+U 1 1 5749308D
+P 6150 3300
+F 0 "R?" V 6230 3300 50  0000 C CNN
+F 1 "50k" V 6150 3300 50  0000 C CNN
+F 2 "" V 6080 3300 50  0000 C CNN
+F 3 "" H 6150 3300 50  0000 C CNN
+	1    6150 3300
+	0    1    1    0
+$EndComp
+Wire Wire Line
+	6400 3450 6400 3300
+Wire Wire Line
+	6400 3300 6300 3300
+Wire Wire Line
+	6000 3300 5850 3300
+Wire Wire Line
+	3050 3300 3200 3300
 $EndSCHEMATC
