File: Placa/Sensores.sch (KiCad schematic (older format))
At the start: 18 parts

Commit message: Avances sobre la placa.
Parts:
- added Q1, Q2: BC548, TO_SOT_Packages_THT:TO-92_Inline_Narrow_Oval, symbol BC548
- added R8, R9: R, Resistors_SMD:R_0805, symbol R
- R10, R11, R12, R13, R14, R15, R16, R17, R18, R19, R20, R21: renamed from R?; footprint (none) -> Resistors_SMD:R_0805
- U3, U4, U5, U6, U7, U8: renamed from U?; footprint TCRT1000 -> tcrt1000:TCRT1000
Connections:
- net labels added: Habilitador1, Habilitador2, habilitado, habilitado2
- wire segments 66 -> 74

Commit message: Modificaciones a la placa
Parts:
- added R28: 180, Resistors_SMD:R_0805, symbol R
- added R32: 33k, Resistors_SMD:R_0805, symbol R
- added U12: TCRT1000, tcrt1000:TCRT1000, symbol TCRT1000
Connections:
- net labels added: Habilitador, Sensor7
- net labels removed: Habilitador1, Habilitador2
- wire segments 74 -> 85

Commit message: se termino el esquematico y asociacion de componentes, falta acomodar y rutear PCB
Parts:
- R8, R9: value R -> 2k2
Changed lines of the file:
@@
 $Descr A4 11693 8268
 encoding utf-8
-Sheet 2 4
+Sheet 4 4
 Title ""
 Date ""
@@
 P 1700 3000
 F 0 "R8" V 1780 3000 50  0000 C CNN
-F 1 "R" V 1700 3000 50  0000 C CNN
+F 1 "2k2" V 1700 3000 50  0000 C CNN
 F 2 "Resistors_SMD:R_0805" V 1630 3000 50  0001 C CNN
 F 3 "" H 1700 3000 50  0000 C CNN
@@
 P 1700 4300
 F 0 "R9" V 1780 4300 50  0000 C CNN
-F 1 "R" V 1700 4300 50  0000 C CNN
+F 1 "2k2" V 1700 4300 50  0000 C CNN
 F 2 "Resistors_SMD:R_0805" V 1630 4300 50  0001 C CNN
 F 3 "" H 1700 4300 50  0000 C CNN

Commit message: Está todo ruteado, falta engrozar pistas, chequear wiki y un chequeo general
Parts:
- R8, R9: footprint Resistors_SMD:R_0805 -> Resistors_ThroughHole:Resistor_Horizontal_RM7mm
- U12, U8: footprint tcrt1000:TCRT1000 -> Pin_Headers:Pin_Header_Straight_1x04
Changed lines of the file:
@@
 F 0 "U8" H 7050 4050 60  0000 C CNN
 F 1 "TCRT1000" H 7300 4250 60  0000 C CNN
-F 2 "tcrt1000:TCRT1000" H 6800 4250 60  0001 C CNN
+F 2 "Pin_Headers:Pin_Header_Straight_1x04" H 6800 4250 60  0001 C CNN
 F 3 "" H 7050 4050 60  0000 C CNN
 	1    7050 4050
@@
 	1    0    0    -1
 $EndComp
+Text HLabel 7950 4550 0    60   Input ~ 0
+Sensor1
 Text HLabel 4850 3100 0    60   Input ~ 0
-Sensor1
+Sensor2
+Text HLabel 4900 4550 0    60   Input ~ 0
+Sensor3
+Text HLabel 7950 3100 0    60   Input ~ 0
+Sensor6
 Text HLabel 6450 3100 0    60   Input ~ 0
-Sensor2
-Text HLabel 7950 3100 0    60   Input ~ 0
-Sensor3
-Text HLabel 7950 4550 0    60   Input ~ 0
-Sensor6
+Sensor5
 Text HLabel 6400 4550 0    60   Input ~ 0
-Sensor5
-Text HLabel 4900 4550 0    60   Input ~ 0
 Sensor4
 Text HLabel 7750 3350 2    60   Input ~ 0
@@
 F 0 "R8" V 1780 3000 50  0000 C CNN
 F 1 "2k2" V 1700 3000 50  0000 C CNN
-F 2 "Resistors_SMD:R_0805" V 1630 3000 50  0001 C CNN
+F 2 "Resistors_ThroughHole:Resistor_Horizontal_RM7mm" V 1630 3000 50  0001 C CNN
 F 3 "" H 1700 3000 50  0000 C CNN
 	1    1700 3000
@@
 Text Label 2250 3300 0    60   ~ 0
 habilitado
-Text Label 3300 2850 2    60   ~ 0
+Text Label 8000 4300 2    60   ~ 0
 habilitado
 Text Label 4900 2850 2    60   ~ 0
@@
 habilitado2
 Text Label 4850 4300 2    60   ~ 0
-habilitado2
+habilitado
 Text Label 6400 4300 2    60   ~ 0
 habilitado2
@@
 F 0 "R9" V 1780 4300 50  0000 C CNN
 F 1 "2k2" V 1700 4300 50  0000 C CNN
-F 2 "Resistors_SMD:R_0805" V 1630 4300 50  0001 C CNN
+F 2 "Resistors_ThroughHole:Resistor_Horizontal_RM7mm" V 1630 4300 50  0001 C CNN
 F 3 "" H 1700 4300 50  0000 C CNN
 	1    1700 4300
@@
 F 0 "U12" H 8650 4050 60  0000 C CNN
 F 1 "TCRT1000" H 8900 4250 60  0000 C CNN
-F 2 "tcrt1000:TCRT1000" H 8400 4250 60  0001 C CNN
+F 2 "Pin_Headers:Pin_Header_Straight_1x04" H 8400 4250 60  0001 C CNN
 F 3 "" H 8650 4050 60  0000 C CNN
 	1    8650 4050
@@
 Wire Wire Line
 	9550 4500 9550 4550
-Text Label 8000 4300 2    60   ~ 0
+Text Label 3300 2850 2    60   ~ 0
 habilitado2
 Wire Wire Line
