File: Placa/Alimentacion.sch (KiCad schematic (older format))
At the start: 16 parts

Commit message: Avances sobre la placa.
Parts:
- C10, C11, C7, C9: renamed from C?; footprint (none) -> Capacitors_ThroughHole:C_Radial_D5_L11_P2.5
- C12, C8: renamed from C?; footprint (none) -> Capacitors_SMD:C_0805_HandSoldering
- JP1: renamed from JP?; footprint (none) -> Pin_Headers:Pin_Header_Straight_2x01
- P10, P11: renamed from P?; footprint (none) -> Pin_Headers:Pin_Header_Straight_1x02
- P8, P9: renamed from P?; footprint (none) -> Pin_Headers:Pin_Header_Straight_1x03
- R22, R23, R24: renamed from R?; footprint (none) -> Resistors_SMD:R_0805
- U10: renamed from U?; footprint TO-220 -> TO_SOT_Packages_THT:TO-220_Neutral123_Vertical
- U9: renamed from U?; footprint (none) -> SOT223-5:SOT223-5

Commit message: estan casi todas las cosas en su lugar, falta cambiar DVRs y regulador y rutear
Parts:
- C8: value 0.1u -> 100n
Changed lines of the file:
@@
 	3900 3750 4250 3750
 $Comp
-L PWR_FLAG #FLG049
+L PWR_FLAG #FLG2
 U 1 1 571B3C7B
 P 4100 3800
-F 0 "#FLG049" H 4100 3895 50  0001 C CNN
+F 0 "#FLG2" H 4100 3895 50  0001 C CNN
 F 1 "PWR_FLAG" H 4100 3980 50  0000 C CNN
 F 2 "" H 4100 3800 50  0000 C CNN
@@
 $EndComp
 $Comp
-L GND #PWR050
+L GND #PWR48
 U 1 1 571B3C8A
 P 5200 2400
-F 0 "#PWR050" H 5200 2150 50  0001 C CNN
+F 0 "#PWR48" H 5200 2150 50  0001 C CNN
 F 1 "GND" H 5200 2250 50  0000 C CNN
 F 2 "" H 5200 2400 50  0000 C CNN
@@
 	8250 3250 8250 3350
 $Comp
-L GND #PWR051
+L GND #PWR53
 U 1 1 571B3CDB
 P 8250 3350
-F 0 "#PWR051" H 8250 3100 50  0001 C CNN
+F 0 "#PWR53" H 8250 3100 50  0001 C CNN
 F 1 "GND" H 8250 3200 50  0000 C CNN
 F 2 "" H 8250 3350 50  0000 C CNN
@@
 	6250 1750 6250 1850
 $Comp
-L GND #PWR052
+L GND #PWR51
 U 1 1 571B3CF2
 P 6250 1850
-F 0 "#PWR052" H 6250 1600 50  0001 C CNN
+F 0 "#PWR51" H 6250 1600 50  0001 C CNN
 F 1 "GND" H 6250 1700 50  0000 C CNN
 F 2 "" H 6250 1850 50  0000 C CNN
@@
 	5950 2100 5950 2000
 $Comp
-L +8V #PWR053
+L +8V #PWR50
 U 1 1 571B3CFC
 P 5950 2000
-F 0 "#PWR053" H 5950 1850 50  0001 C CNN
+F 0 "#PWR50" H 5950 1850 50  0001 C CNN
 F 1 "+8V" H 5950 2140 50  0000 C CNN
 F 2 "" H 5950 2000 50  0000 C CNN
@@
 $EndComp
 $Comp
-L GND #PWR054
+L GND #PWR49
 U 1 1 571B3D13
 P 5800 2550
-F 0 "#PWR054" H 5800 2300 50  0001 C CNN
+F 0 "#PWR49" H 5800 2300 50  0001 C CNN
 F 1 "GND" H 5800 2400 50  0000 C CNN
 F 2 "" H 5800 2550 50  0000 C CNN
@@
 P 4700 2350
 F 0 "C8" H 4725 2450 50  0000 L CNN
-F 1 "0.1u" H 4725 2250 50  0000 L CNN
+F 1 "100n" H 4725 2250 50  0000 L CNN
 F 2 "Capacitors_SMD:C_0805_HandSoldering" H 4738 2200 50  0001 C CNN
 F 3 "" H 4700 2350 50  0000 C CNN
@@
 Connection ~ 4550 2550
 $Comp
-L GND #PWR055
+L GND #PWR46
 U 1 1 571B3D2E
 P 4550 2600
-F 0 "#PWR055" H 4550 2350 50  0001 C CNN
+F 0 "#PWR46" H 4550 2350 50  0001 C CNN
 F 1 "GND" H 4550 2450 50  0000 C CNN
 F 2 "" H 4550 2600 50  0000 C CNN
@@
 Connection ~ 8700 2200
 $Comp
-L GND #PWR056
+L GND #PWR54
 U 1 1 571B3D56
 P 8700 2250
-F 0 "#PWR056" H 8700 2000 50  0001 C CNN
+F 0 "#PWR54" H 8700 2000 50  0001 C CNN
 F 1 "GND" H 8700 2100 50  0000 C CNN
 F 2 "" H 8700 2250 50  0000 C CNN
@@
 	7050 2150 7050 2250
 $Comp
-L GND #PWR057
+L GND #PWR52
 U 1 1 571B3D5F
 P 7050 2250
-F 0 "#PWR057" H 7050 2000 50  0001 C CNN
+F 0 "#PWR52" H 7050 2000 50  0001 C CNN
 F 1 "GND" H 7050 2100 50  0000 C CNN
 F 2 "" H 7050 2250 50  0000 C CNN
@@
 	5150 3750 5150 3800
 $Comp
-L GND #PWR058
+L GND #PWR47
 U 1 1 571B4008
 P 5150 3800
-F 0 "#PWR058" H 5150 3550 50  0001 C CNN
+F 0 "#PWR47" H 5150 3550 50  0001 C CNN
 F 1 "GND" H 5150 3650 50  0000 C CNN
 F 2 "" H 5150 3800 50  0000 C CNN
@@
 Connection ~ 5150 3650
 $Comp
-L PWR_FLAG #FLG059
+L PWR_FLAG #FLG3
 U 1 1 571B4012
 P 4950 3550
-F 0 "#FLG059" H 4950 3645 50  0001 C CNN
+F 0 "#FLG3" H 4950 3645 50  0001 C CNN
 F 1 "PWR_FLAG" H 4950 3730 50  0000 C CNN
 F 2 "" H 4950 3550 50  0000 C CNN
@@
 $EndComp
 $Comp
-L PWR_FLAG #FLG060
+L PWR_FLAG #FLG4
 U 1 1 571B4018
 P 4950 3850
-F 0 "#FLG060" H 4950 3945 50  0001 C CNN
+F 0 "#FLG4" H 4950 3945 50  0001 C CNN
 F 1 "PWR_FLAG" H 4950 4030 50  0000 C CNN
 F 2 "" H 4950 3850 50  0000 C CNN
@@
 Connection ~ 4300 1950
 $Comp
-L PWR_FLAG #FLG061
+L PWR_FLAG #FLG1
 U 1 1 572E1B30
 P 4050 1950
-F 0 "#FLG061" H 4050 2045 50  0001 C CNN
+F 0 "#FLG1" H 4050 2045 50  0001 C CNN
 F 1 "PWR_FLAG" H 4050 2130 50  0000 C CNN
 F 2 "" H 4050 1950 50  0000 C CNN

Commit message: Modificaciones a la placa
Parts:
- removed P11: CONN_01X02, Pin_Headers:Pin_Header_Straight_1x02, symbol CONN_01X02
- removed P8: CONN_01X03, Pin_Headers:Pin_Header_Straight_1x03, symbol CONN_01X03
Connections:
- net +8v is gone; now on net Vbat: P9.3 (P3), U9.1 (Vin)
- net Vreg is gone; now on net Vbat: C10.1, U10.3 (IN)
- net +8V renamed Vbat
Other:
- note added: "Al conectar el jumper regula 6 V,\nsi se lo desconecta regula 9 V"
- note removed: "Conector segunda bateria\n"
- note removed: "Selector 2 o 3 celdas"
Changed lines of the file:
@@
 LIBS:reg_204-5
 LIBS:DVR8833
+LIBS:sn74lvc2g86
+LIBS:placa-cache
 EELAYER 25 0
 EELAYER END
 $Descr A4 11693 8268
 encoding utf-8
-Sheet 4 4
+Sheet 3 4
 Title ""
 Date ""
@@
 	3900 3750 4250 3750
 $Comp
-L PWR_FLAG #FLG2
+L PWR_FLAG #FLG047
 U 1 1 571B3C7B
 P 4100 3800
-F 0 "#FLG2" H 4100 3895 50  0001 C CNN
+F 0 "#FLG047" H 4100 3895 50  0001 C CNN
 F 1 "PWR_FLAG" H 4100 3980 50  0000 C CNN
 F 2 "" H 4100 3800 50  0000 C CNN
@@
 $EndComp
 $Comp
-L GND #PWR48
+L GND #PWR048
 U 1 1 571B3C8A
 P 5200 2400
-F 0 "#PWR48" H 5200 2150 50  0001 C CNN
+F 0 "#PWR048" H 5200 2150 50  0001 C CNN
 F 1 "GND" H 5200 2250 50  0000 C CNN
 F 2 "" H 5200 2400 50  0000 C CNN
@@
 	8250 3250 8250 3350
 $Comp
-L GND #PWR53
+L GND #PWR049
 U 1 1 571B3CDB
 P 8250 3350
-F 0 "#PWR53" H 8250 3100 50  0001 C CNN
+F 0 "#PWR049" H 8250 3100 50  0001 C CNN
 F 1 "GND" H 8250 3200 50  0000 C CNN
 F 2 "" H 8250 3350 50  0000 C CNN
@@
 	6250 1750 6250 1850
 $Comp
-L GND #PWR51
+L GND #PWR050
 U 1 1 571B3CF2
 P 6250 1850
-F 0 "#PWR51" H 6250 1600 50  0001 C CNN
+F 0 "#PWR050" H 6250 1600 50  0001 C CNN
 F 1 "GND" H 6250 1700 50  0000 C CNN
 F 2 "" H 6250 1850 50  0000 C CNN
@@
 Wire Wire Line
 	5950 2100 5950 2000
-$Comp
-L +8V #PWR50
-U 1 1 571B3CFC
-P 5950 2000
-F 0 "#PWR50" H 5950 1850 50  0001 C CNN
-F 1 "+8V" H 5950 2140 50  0000 C CNN
-F 2 "" H 5950 2000 50  0000 C CNN
-F 3 "" H 5950 2000 50  0000 C CNN
-	1    5950 2000
-	1    0    0    -1
-$EndComp
 $Comp
 L CP C7
@@
 $EndComp
 $Comp
-L GND #PWR49
+L GND #PWR051
 U 1 1 571B3D13
 P 5800 2550
-F 0 "#PWR49" H 5800 2300 50  0001 C CNN
+F 0 "#PWR051" H 5800 2300 50  0001 C CNN
 F 1 "GND" H 5800 2400 50  0000 C CNN
 F 2 "" H 5800 2550 50  0000 C CNN
@@
 Connection ~ 4550 2550
 $Comp
-L GND #PWR46
+L GND #PWR052
 U 1 1 571B3D2E
 P 4550 2600
-F 0 "#PWR46" H 4550 2350 50  0001 C CNN
+F 0 "#PWR052" H 4550 2350 50  0001 C CNN
 F 1 "GND" H 4550 2450 50  0000 C CNN
 F 2 "" H 4550 2600 50  0000 C CNN
@@
 Connection ~ 8700 2200
 $Comp
-L GND #PWR54
+L GND #PWR053
 U 1 1 571B3D56
 P 8700 2250
-F 0 "#PWR54" H 8700 2000 50  0001 C CNN
+F 0 "#PWR053" H 8700 2000 50  0001 C CNN
 F 1 "GND" H 8700 2100 50  0000 C CNN
 F 2 "" H 8700 2250 50  0000 C CNN
@@
 	7050 2150 7050 2250
 $Comp
-L GND #PWR52
+L GND #PWR054
 U 1 1 571B3D5F
 P 7050 2250
-F 0 "#PWR52" H 7050 2000 50  0001 C CNN
+F 0 "#PWR054" H 7050 2000 50  0001 C CNN
 F 1 "GND" H 7050 2100 50  0000 C CNN
 F 2 "" H 7050 2250 50  0000 C CNN
@@
 	5150 3750 5150 3800
 $Comp
-L GND #PWR47
+L GND #PWR055
 U 1 1 571B4008
 P 5150 3800
-F 0 "#PWR47" H 5150 3550 50  0001 C CNN
+F 0 "#PWR055" H 5150 3550 50  0001 C CNN
 F 1 "GND" H 5150 3650 50  0000 C CNN
 F 2 "" H 5150 3800 50  0000 C CNN
@@
 Connection ~ 5150 3650
 $Comp
-L PWR_FLAG #FLG3
+L PWR_FLAG #FLG056
 U 1 1 571B4012
 P 4950 3550
-F 0 "#FLG3" H 4950 3645 50  0001 C CNN
+F 0 "#FLG056" H 4950 3645 50  0001 C CNN
 F 1 "PWR_FLAG" H 4950 3730 50  0000 C CNN
 F 2 "" H 4950 3550 50  0000 C CNN
@@
 $EndComp
 $Comp
-L PWR_FLAG #FLG4
+L PWR_FLAG #FLG057
 U 1 1 571B4018
 P 4950 3850
-F 0 "#FLG4" H 4950 3945 50  0001 C CNN
+F 0 "#FLG057" H 4950 3945 50  0001 C CNN
 F 1 "PWR_FLAG" H 4950 4030 50  0000 C CNN
 F 2 "" H 4950 3850 50  0000 C CNN
@@
 	-1   0    0    1
 $EndComp
-$Comp
-L CONN_01X02 P11
-U 1 1 571B401E
-P 5500 4750
-F 0 "P11" H 5500 4900 50  0000 C CNN
-F 1 "CONN_01X02" V 5600 4750 50  0000 C CNN
-F 2 "Pin_Headers:Pin_Header_Straight_1x02" H 5500 4750 50  0001 C CNN
-F 3 "" H 5500 4750 50  0000 C CNN
-	1    5500 4750
-	1    0    0    -1
-$EndComp
-$Comp
-L CONN_01X03 P8
-U 1 1 571B4035
-P 4400 4750
-F 0 "P8" H 4400 4950 50  0000 C CNN
-F 1 "CONN_01X03" V 4500 4750 50  0000 C CNN
-F 2 "Pin_Headers:Pin_Header_Straight_1x03" H 4400 4750 50  0001 C CNN
-F 3 "" H 4400 4750 50  0000 C CNN
-	1    4400 4750
-	1    0    0    -1
-$EndComp
 Text HLabel 8500 1650 2    60   Input ~ 0
 Vmot
-Wire Wire Line
-	4000 4750 4200 4750
-Wire Wire Line
-	4000 4850 4200 4850
-Wire Wire Line
-	4200 4650 3950 4650
-Text Label 5050 4700 0    60   ~ 0
-+12V
-Wire Wire Line
-	5050 4700 5300 4700
-Wire Wire Line
-	5100 4800 5300 4800
 Text HLabel 5150 3450 2    60   Input ~ 0
 +Batt
@@
 +Batt
 Text Label 3900 3750 0    60   ~ 0
-+8v
-Text Label 5100 4800 0    60   ~ 0
-+8v
-Text Label 4000 4850 0    60   ~ 0
-+8v
-Text Label 3950 4650 0    60   ~ 0
-+12V
-Text Label 4000 4750 0    60   ~ 0
-Vreg
+Vbat
 Text Label 6950 1650 0    60   ~ 0
-Vreg
+Vbat
 Text HLabel 4300 1700 0    60   Input ~ 0
 +5V
 Text Label 4500 1600 0    60   ~ 0
-+8v
-Text Notes 4900 4450 0    60   ~ 0
-Conector segunda bateria\n
-Text Notes 3750 4450 0    60   ~ 0
-Selector 2 o 3 celdas
+Vbat
 Text Notes 4700 3200 0    60   ~ 0
 Conector primera bateria
@@
 Connection ~ 4300 1950
 $Comp
-L PWR_FLAG #FLG1
+L PWR_FLAG #FLG058
 U 1 1 572E1B30
 P 4050 1950
-F 0 "#FLG1" H 4050 2045 50  0001 C CNN
+F 0 "#FLG058" H 4050 2045 50  0001 C CNN
 F 1 "PWR_FLAG" H 4050 2130 50  0000 C CNN
 F 2 "" H 4050 1950 50  0000 C CNN
@@
 $EndComp
 Connection ~ 8400 1750
+Text Notes 7300 3750 0    60   ~ 0
+Al conectar el jumper regula 6 V,\nsi se lo desconecta regula 9 V
+Text Label 5950 2000 0    60   ~ 0
+Vbat
 $EndSCHEMATC

Commit message: Está todo ruteado, falta engrozar pistas, chequear wiki y un chequeo general
Parts:
- C10, C11, C7, C9: footprint Capacitors_ThroughHole:C_Radial_D5_L11_P2.5 -> Capacitors_SMD:C_0805_HandSoldering
Changed lines of the file:
@@
 F 0 "C7" H 4425 2450 50  0000 L CNN
 F 1 "10u" H 4425 2250 50  0000 L CNN
-F 2 "Capacitors_ThroughHole:C_Radial_D5_L11_P2.5" H 4438 2200 50  0001 C CNN
+F 2 "Capacitors_SMD:C_0805_HandSoldering" H 4438 2200 50  0001 C CNN
 F 3 "" H 4400 2350 50  0000 C CNN
 	1    4400 2350
@@
 F 0 "C9" H 5825 2450 50  0000 L CNN
 F 1 "10u" H 5825 2250 50  0000 L CNN
-F 2 "Capacitors_ThroughHole:C_Radial_D5_L11_P2.5" H 5838 2200 50  0001 C CNN
+F 2 "Capacitors_SMD:C_0805_HandSoldering" H 5838 2200 50  0001 C CNN
 F 3 "" H 5800 2350 50  0000 C CNN
 	1    5800 2350
@@
 F 0 "C10" H 7075 2100 50  0000 L CNN
 F 1 "10u" H 7075 1900 50  0000 L CNN
-F 2 "Capacitors_ThroughHole:C_Radial_D5_L11_P2.5" H 7088 1850 50  0001 C CNN
+F 2 "Capacitors_SMD:C_0805_HandSoldering" H 7088 1850 50  0001 C CNN
 F 3 "" H 7050 2000 50  0000 C CNN
 	1    7050 2000
@@
 F 0 "C11" H 8575 2100 50  0000 L CNN
 F 1 "10u" H 8575 1900 50  0000 L CNN
-F 2 "Capacitors_ThroughHole:C_Radial_D5_L11_P2.5" H 8588 1850 50  0001 C CNN
+F 2 "Capacitors_SMD:C_0805_HandSoldering" H 8588 1850 50  0001 C CNN
 F 3 "" H 8550 2000 50  0000 C CNN
 	1    8550 2000

Commit message: Se termino la placa, y se mando a fabricar.
Parts:
- C10, C11, C7, C9: footprint Capacitors_SMD:C_0805_HandSoldering -> Capacitors_SMD:C_1206
- P10: footprint Pin_Headers:Pin_Header_Straight_1x02 -> Connectors_Molex:Molex_KK-6410-02_02x2.54mm_Straight
Changed lines of the file:
@@
 LIBS:DVR8833
 LIBS:sn74lvc2g86
+LIBS:logo
 LIBS:placa-cache
 EELAYER 25 0
@@
 F 0 "C7" H 4425 2450 50  0000 L CNN
 F 1 "10u" H 4425 2250 50  0000 L CNN
-F 2 "Capacitors_SMD:C_0805_HandSoldering" H 4438 2200 50  0001 C CNN
+F 2 "Capacitors_SMD:C_1206" H 4438 2200 50  0001 C CNN
 F 3 "" H 4400 2350 50  0000 C CNN
 	1    4400 2350
@@
 F 0 "C9" H 5825 2450 50  0000 L CNN
 F 1 "10u" H 5825 2250 50  0000 L CNN
-F 2 "Capacitors_SMD:C_0805_HandSoldering" H 5838 2200 50  0001 C CNN
+F 2 "Capacitors_SMD:C_1206" H 5838 2200 50  0001 C CNN
 F 3 "" H 5800 2350 50  0000 C CNN
 	1    5800 2350
@@
 F 0 "C10" H 7075 2100 50  0000 L CNN
 F 1 "10u" H 7075 1900 50  0000 L CNN
-F 2 "Capacitors_SMD:C_0805_HandSoldering" H 7088 1850 50  0001 C CNN
+F 2 "Capacitors_SMD:C_1206" H 7088 1850 50  0001 C CNN
 F 3 "" H 7050 2000 50  0000 C CNN
 	1    7050 2000
@@
 F 0 "C11" H 8575 2100 50  0000 L CNN
 F 1 "10u" H 8575 1900 50  0000 L CNN
-F 2 "Capacitors_SMD:C_0805_HandSoldering" H 8588 1850 50  0001 C CNN
+F 2 "Capacitors_SMD:C_1206" H 8588 1850 50  0001 C CNN
 F 3 "" H 8550 2000 50  0000 C CNN
 	1    8550 2000
@@
 F 0 "P10" H 5450 3850 50  0000 C CNN
 F 1 "CONN_01X02" V 5550 3700 50  0000 C CNN
-F 2 "Pin_Headers:Pin_Header_Straight_1x02" H 5450 3700 50  0001 C CNN
+F 2 "Connectors_Molex:Molex_KK-6410-02_02x2.54mm_Straight" H 5450 3700 50  0001 C CNN
 F 3 "" H 5450 3700 50  0000 C CNN
 	1    5450 3700

Commit message: Agrego cambios sugeridos en la wiki de github.
Parts:
- added C14: 0.01uF, Capacitors_SMD:C_0805, symbol C
Connections:
- net GND: now also C14.2; no longer U9.4 (NR)
- new net: C14.1, U9.4 (NR)
Changed lines of the file:
@@
 LIBS:DVR8833
 LIBS:sn74lvc2g86
-LIBS:logo
-LIBS:placa-cache
 EELAYER 25 0
 EELAYER END
@@
 	3900 3750 4250 3750
 $Comp
-L PWR_FLAG #FLG047
+L PWR_FLAG #FLG048
 U 1 1 571B3C7B
 P 4100 3800
-F 0 "#FLG047" H 4100 3895 50  0001 C CNN
+F 0 "#FLG048" H 4100 3895 50  0001 C CNN
 F 1 "PWR_FLAG" H 4100 3980 50  0000 C CNN
 F 2 "" H 4100 3800 50  0000 C CNN
@@
 $EndComp
 $Comp
-L GND #PWR048
+L GND #PWR049
 U 1 1 571B3C8A
 P 5200 2400
-F 0 "#PWR048" H 5200 2150 50  0001 C CNN
+F 0 "#PWR049" H 5200 2150 50  0001 C CNN
 F 1 "GND" H 5200 2250 50  0000 C CNN
 F 2 "" H 5200 2400 50  0000 C CNN
@@
 	8250 3250 8250 3350
 $Comp
-L GND #PWR049
+L GND #PWR050
 U 1 1 571B3CDB
 P 8250 3350
-F 0 "#PWR049" H 8250 3100 50  0001 C CNN
+F 0 "#PWR050" H 8250 3100 50  0001 C CNN
 F 1 "GND" H 8250 3200 50  0000 C CNN
 F 2 "" H 8250 3350 50  0000 C CNN
@@
 	5700 1750 6250 1750
 Wire Wire Line
-	6250 1750 6250 1850
-$Comp
-L GND #PWR050
+	6250 1750 6250 1900
+$Comp
+L GND #PWR051
 U 1 1 571B3CF2
-P 6250 1850
-F 0 "#PWR050" H 6250 1600 50  0001 C CNN
-F 1 "GND" H 6250 1700 50  0000 C CNN
-F 2 "" H 6250 1850 50  0000 C CNN
-F 3 "" H 6250 1850 50  0000 C CNN
-	1    6250 1850
+P 6250 2250
+F 0 "#PWR051" H 6250 2000 50  0001 C CNN
+F 1 "GND" H 6250 2100 50  0000 C CNN
+F 2 "" H 6250 2250 50  0000 C CNN
+F 3 "" H 6250 2250 50  0000 C CNN
+	1    6250 2250
 	1    0    0    -1
 $EndComp
@@
 $EndComp
 $Comp
-L GND #PWR051
+L GND #PWR052
 U 1 1 571B3D13
 P 5800 2550
-F 0 "#PWR051" H 5800 2300 50  0001 C CNN
+F 0 "#PWR052" H 5800 2300 50  0001 C CNN
 F 1 "GND" H 5800 2400 50  0000 C CNN
 F 2 "" H 5800 2550 50  0000 C CNN
@@
 Connection ~ 4550 2550
 $Comp
-L GND #PWR052
+L GND #PWR053
 U 1 1 571B3D2E
 P 4550 2600
-F 0 "#PWR052" H 4550 2350 50  0001 C CNN
+F 0 "#PWR053" H 4550 2350 50  0001 C CNN
 F 1 "GND" H 4550 2450 50  0000 C CNN
 F 2 "" H 4550 2600 50  0000 C CNN
@@
 Connection ~ 8700 2200
 $Comp
-L GND #PWR053
+L GND #PWR054
 U 1 1 571B3D56
 P 8700 2250
-F 0 "#PWR053" H 8700 2000 50  0001 C CNN
+F 0 "#PWR054" H 8700 2000 50  0001 C CNN
 F 1 "GND" H 8700 2100 50  0000 C CNN
 F 2 "" H 8700 2250 50  0000 C CNN
@@
 	7050 2150 7050 2250
 $Comp
-L GND #PWR054
+L GND #PWR055
 U 1 1 571B3D5F
 P 7050 2250
-F 0 "#PWR054" H 7050 2000 50  0001 C CNN
+F 0 "#PWR055" H 7050 2000 50  0001 C CNN
 F 1 "GND" H 7050 2100 50  0000 C CNN
 F 2 "" H 7050 2250 50  0000 C CNN
@@
 	5150 3750 5150 3800
 $Comp
-L GND #PWR055
+L GND #PWR056
 U 1 1 571B4008
 P 5150 3800
-F 0 "#PWR055" H 5150 3550 50  0001 C CNN
+F 0 "#PWR056" H 5150 3550 50  0001 C CNN
 F 1 "GND" H 5150 3650 50  0000 C CNN
 F 2 "" H 5150 3800 50  0000 C CNN
@@
 Connection ~ 5150 3650
 $Comp
-L PWR_FLAG #FLG056
+L PWR_FLAG #FLG057
 U 1 1 571B4012
 P 4950 3550
-F 0 "#FLG056" H 4950 3645 50  0001 C CNN
+F 0 "#FLG057" H 4950 3645 50  0001 C CNN
 F 1 "PWR_FLAG" H 4950 3730 50  0000 C CNN
 F 2 "" H 4950 3550 50  0000 C CNN
@@
 $EndComp
 $Comp
-L PWR_FLAG #FLG057
+L PWR_FLAG #FLG058
 U 1 1 571B4018
 P 4950 3850
-F 0 "#FLG057" H 4950 3945 50  0001 C CNN
+F 0 "#FLG058" H 4950 3945 50  0001 C CNN
 F 1 "PWR_FLAG" H 4950 4030 50  0000 C CNN
 F 2 "" H 4950 3850 50  0000 C CNN
@@
 Connection ~ 4300 1950
 $Comp
-L PWR_FLAG #FLG058
+L PWR_FLAG #FLG059
 U 1 1 572E1B30
 P 4050 1950
-F 0 "#FLG058" H 4050 2045 50  0001 C CNN
+F 0 "#FLG059" H 4050 2045 50  0001 C CNN
 F 1 "PWR_FLAG" H 4050 2130 50  0000 C CNN
 F 2 "" H 4050 1950 50  0000 C CNN
@@
 Text Label 5950 2000 0    60   ~ 0
 Vbat
+$Comp
+L C C14
+U 1 1 58547F78
+P 6250 2050
+F 0 "C14" H 6275 2150 50  0000 L CNN
+F 1 "0.01uF" H 6275 1950 50  0000 L CNN
+F 2 "Capacitors_SMD:C_0805" H 6288 1900 50  0001 C CNN
+F 3 "" H 6250 2050 50  0000 C CNN
+	1    6250 2050
+	1    0    0    -1
+$EndComp
+Wire Wire Line
+	6250 2200 6250 2250
 $EndSCHEMATC
